Commit message: Fix camera to base link transform

File: src/sentry_realsense/urdf/mount.urdf.xacro (robot description, xacro)
@@ -1,10 +1,10 @@
 <?xml version="1.0" ?>
-<robot xmlns:xacro="http://www.ros.org/wiki/xacro">
+<robot name="husky" xmlns:xacro="http://www.ros.org/wiki/xacro">
+    <link name="base_link"></link>
+    <link name="rs_camera_link"></link>
     <joint name="mount_joint" type="fixed">
         <origin xyz="0.3984752 0 0.2638552" rpy="0 0 0" />
         <parent link="base_link"/>
-        <child link="camera_link" />
+        <child link="rs_camera_link" />
     </joint>
-    <link name="camera_link">
-    </link>
 </robot>
