Commit message: Reverse LIDAR direction in URDF

File: src/sentry_mapper/urdf/lidar.urdf.xacro (robot description, xacro)
@@ -4,5 +4,5 @@
     <link name="laser_frame"></link>
     <joint name="lidar_joint" type="fixed">
-        <origin xyz="0.3984752 0 0.2638552" rpy="0 0 0" />
+        <origin xyz="0.3984752 0 0.2638552" rpy="0 0 ${pi}" />
         <parent link="base_link"/>
         <child link="laser_frame" />
